Commit message: Big maj with modification done for experiment -- servo, focus_curve -- MAIS ws pas à jour par rapport à UR10e : TODO

File: src/icube_ur_cell/icube_ur_cell_control/urdf/icube_ur_cell_ros2_control.urdf.xacro (robot description, xacro)
@@ -6,5 +6,5 @@
   <xacro:include filename="$(find ur_description)/urdf/ur.ros2_control.xacro"/>
   <!--We need to specify the arguments used for parametrizing our description-->
-  <xacro:arg name="ur_type" default="ur5e"/>
+  <xacro:arg name="ur_type" default="ur5"/>
   <xacro:arg name="joint_limit_parameters_file" default="$(find ur_description)/config/$(arg ur_type)/joint_limits.yaml"/>
   <xacro:arg name="kinematics_parameters_file" default="$(find ur_description)/config/$(arg ur_type)/default_kinematics.yaml"/>

File: src/icube_ur_cell/icube_ur_cell_description/urdf/icube_ur_cell_macro.xacro (robot description, xacro)
@@ -34,4 +34,38 @@
     <child link="ground_plane"/>
   </joint>
+  <link name="support_ur">
+    <visual>
+      <origin rpy="0 0 0" xyz="0 0 0"/>
+      <geometry>
+        <box size="0.7 0.65 1.0"/>
+      </geometry>
+      <material name="ground_white">
+        <color rgba="1 1 1 0.5"/>
+      </material>
+    </visual>
+    <collision>
+      <origin rpy="0.0 0.0 0" xyz="0 0 0"/>
+      <geometry>
+        <box size="0.7 0.65 1.0"/>
+      </geometry>
+    </collision>
+  </link>
+  <joint name="support_ur_joint" type="fixed">
+    <origin xyz="0 0 0.5" rpy="0 0 0"/>
+    <parent link="ground_plane"/>
+    <child link="support_ur"/>
+  </joint>
+  <link name="optical_camera_frame"/>
+  <joint name="optical_camera_frame" type="fixed">
+    <origin xyz="0.25 -0.6 1.7" rpy="0 ${pi} ${pi}"/>
+    <parent link="ground_plane"/>
+    <child link="optical_camera_frame"/>
+  </joint>
+  <link name="vimbax_camera_DEV_000F315CCC4E"/>
+  <joint name="optical_vimbax_frame" type="fixed">
+    <origin xyz="0.0 -0.0 0.0" rpy="0 0 0"/>
+    <parent link="optical_camera_frame"/>
+    <child link="vimbax_camera_DEV_000F315CCC4E"/>
+  </joint>
   <!--parent="robot_mount"-->
     <!--This will create the specific robot-->
@@ -39,5 +73,5 @@
       name="${ur_type}"
       tf_prefix="${ur_type}_"
-      parent="ground_plane"
+      parent="support_ur"
       joint_limits_parameters_file="${joint_limits_parameters_file}"
       kinematics_parameters_file="${kinematics_parameters_file}"
@@ -46,5 +80,5 @@
       generate_ros2_control_tag="false"
     >
-      <origin xyz="0 0 0" rpy="0 0 0" />
+      <origin xyz="0 0 0.5" rpy="0 0 0" />
     </xacro:ur_robot>
     <xacro:plate_support

File: src/icube_ur_cell/icube_ur_cell_description/urdf/plate_support_macro.xacro (robot description, xacro)
@@ -48,5 +48,11 @@
       <parent link="${parent}" />
       <child link="${tf_prefix}plate_support" />
-      <origin xyz="0 0 0.0" rpy="0 0 0" />
+      <origin xyz="0 0 0.0" rpy="0 0 ${pi/4}" />
+  </joint>
+<link name="${tf_prefix}target_support"/>
+<joint name="${tf_prefix}target_support_joint" type="fixed">
+      <parent link="${tf_prefix}plate_support" />
+      <child link="${tf_prefix}target_support" />
+      <origin xyz="0 0 0.0" rpy="0 ${pi} 0" />
   </joint>
 </xacro:macro>
